Commit message: add joints

File: articulated.urdf (robot description, URDF)
Before this commit: robot myfirst, 1 links, 0 joints
Links:
- added link elbow; visual box size=0.7 0.18 0.18
- added link shoulder; visual box size=1 0.2 0.2
Joints:
- added joint base_to_shoulder: type fixed, parent base_link, child shoulder, origin xyz=0 0 0.3
- added joint shoulder_to_elbow: type fixed, parent shoulder, child elbow, origin xyz=-0.6 0 0.6

Commit message: finish joints

File: articulated.urdf (robot description, URDF)
Before this commit: robot myfirst, 3 links, 2 joints
Links:
- added link cylinder1; visual cylinder length=0.6 radius=0.2
- link base_link: geometry visual box size=1 1 0.1
Joints:
- removed joint base_to_shoulder
- added joint base_to_cylinder: type revolute, parent base_link, child cylinder1, origin xyz=0 0 0.3, axis 0 0 1, limit lower=0 upper=3 effort=1000.0 velocity=0.5
- added joint cylinder_to_shoulder: type revolute, parent cylinder1, child shoulder, origin xyz=0 0 0.3, axis 0 1 0, limit lower=-0.5 upper=0.5 effort=1000.0 velocity=0.5
- joint shoulder_to_elbow: axis (none) -> 0 1 0; limit (none) -> lower=-0.8 upper=0.8 effort=1000.0 velocity=0.5; type fixed -> revolute
